Commit message: Update login feature

File: src/theimc_description/urdf/theimc.urdf (robot description, URDF)
Before this commit: robot theimcbot_urdf, 8 links, 7 joints
Joints:
- joint imu_joint: origin xyz=0 0 0 rpy=0 0 0 -> xyz=-0.298 0.378 0.147 rpy=0 0 0

Commit message: Update login feature

File: src/theimc_description/urdf/theimc.urdf (robot description, URDF)
Before this commit: robot theimcbot_urdf, 8 links, 7 joints
Links:
- removed link camera_rgb_frame
- added link camera_color_optical_frame
Joints:
- removed joint camera_rgb_joint
- added joint camera_color_optical_joint: type fixed, parent camera_link, child camera_color_optical_frame, origin xyz=0 0 0 rpy=-1.5708 0 -1.5708

Commit message: update

File: src/theimc_description/urdf/theimc.urdf (robot description, URDF)
Before this commit: robot theimcbot_urdf, 8 links, 7 joints
Links:
- removed link camera_color_optical_frame
Joints:
- removed joint camera_color_optical_joint
- joint camera_joint: origin xyz=0.19 0 0.10 rpy=0 0 0 -> xyz=0.41 0 0.10 rpy=0 0 0

Commit message: update

File: src/theimc_description/urdf/theimc.urdf (robot description, URDF)
Before this commit: robot theimcbot_urdf, 7 links, 6 joints
Joints:
- joint base_joint: origin xyz=0.0 0.0 0.33 rpy=0 0 0 -> xyz=0.0 0.0 0.17 rpy=0 0 0
- joint camera_joint: origin xyz=0.41 0 0.10 rpy=0 0 0 -> xyz=0.41 0 0.01 rpy=0 0 0
